File: Hardware/esp_automation/BUZZER.kicad_sch (KiCad schematic)
At the start: 3 parts, among them Q1 2N7002

Commit message: .
Connections:
- net +5V renamed +12V
Changed lines of the file:
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@@
+    )
+  )
+  (symbol (lib_id "power:+12V") (at 42.545 31.75 0) (unit 1)
+    (in_bom yes) (on_board yes) (dnp no) (fields_autoplaced)
+    (property "Reference" "#PWR060" (at 42.545 35.56 0)
+      (effects (font (size 1.27 1.27)) hide)
+    )
+    (property "Value" "+12V" (at 42.545 26.67 0)
+      (effects (font (size 1.27 1.27)))
+    )
+    (property "Footprint" "" (at 42.545 31.75 0)
+      (effects (font (size 1.27 1.27)) hide)
+    )
+    (property "Datasheet" "" (at 42.545 31.75 0)
+      (effects (font (size 1.27 1.27)) hide)
+    )
+    (pin "1")
+    (instances
+      (project "3d_sla_printer"
+        (path "/42e3bda7-42fe-4a9a-b127-3e0d2b22ba14/d8aa4495-6084-4fc3-bfa1-98ba209b054d"
+          (reference "#PWR060") (unit 1)
+        )
+      )
+      (project "esp_automation"
+        (path "/beacb42a-3344-450f-9913-7e99b3038b5c/a33ae25d-c8a0-4eb2-9d87-c713d17e9e55"
+          (reference "#PWR042") (unit 1)
+        )
+        (path "/beacb42a-3344-450f-9913-7e99b3038b5c/fe915d4d-7262-4390-817b-c04a9b0d7da4"
+          (reference "#PWR018") (unit 1)
+        )
+      )
+      (project "Cold_Room_Controller"
+        (path "/ef7b0605-ef7d-4b5f-bcde-eac45c665c82/66d94c9d-33c9-49ba-a394-8f2119977178"
+          (reference "#PWR029") (unit 1)
+        )
+      )
     )
   )
@@
         )
       )
-    )
-  )
-  (symbol (lib_id "power:+5V") (at 42.545 31.75 0) (unit 1)
-    (in_bom yes) (on_board yes) (dnp no)
-    (property "Reference" "#PWR033" (at 42.545 35.56 0)
-      (effects (font (size 1.27 1.27)) hide)
-    )
-    (property "Value" "+5V" (at 42.545 27.94 0)
-      (effects (font (size 1.27 1.27)))
-    )
-    (property "Footprint" "" (at 42.545 31.75 0)
-      (effects (font (size 1.27 1.27)) hide)
-    )
-    (property "Datasheet" "" (at 42.545 31.75 0)
-      (effects (font (size 1.27 1.27)) hide)
-    )
-    (pin "1")
-    (instances
-      (project "esp_automation"
-        (path "/beacb42a-3344-450f-9913-7e99b3038b5c/fe915d4d-7262-4390-817b-c04a9b0d7da4"
-          (reference "#PWR033") (unit 1)
-        )
-      )
