File: Hardware/esp_automation/POWER.kicad_sch (KiCad schematic)
At the start: 20 parts, among them J4 Conn_01x02, T1 Transformer_1P_1S, U3 L7805, U4 AMS1117-3.3

Commit message: .
Parts:
- removed C6: 220UF 25V, Capacitor_SMD:CP_Elec_8x10.5, symbol Device:C_Polarized_Small
- removed D2: Led_Blue, LED_SMD:LED_0805_2012Metric, symbol Device:LED_Small
- removed R4: 330R, Resistor_SMD:R_0805_2012Metric, symbol Device:R_Small_US
- removed U3: L7805, Package_TO_SOT_SMD:TO-252-2, symbol Regulator_Linear:L7812
- added C19: 100nF, Capacitor_SMD:C_0805_2012Metric, symbol Device:C_Small
- added C20: 1000UF 25V SMD, Capacitor_SMD:CP_Elec_10x12.6, symbol Device:C_Polarized_Small
- added D8: SS34, Diode_SMD:D_SMC, symbol Device:D_Schottky
- added L3: 100uH, Inductor_SMD:L_12x12mm_H4.5mm, symbol Device:L_Small
- added U6: LM2576HVS-12, Package_TO_SOT_SMD:TO-263-5_TabPin3, symbol Regulator_Switching:LM2576HVS-12
- D1: footprint Package_TO_SOT_SMD:TO-269AA -> GOFootprint:DB157S
- T1: footprint gkhnmlym:ASLAN220-12VAC -> GOFootprint:ASLAN 151112
Connections:
- net +5V is gone; now on net +12V: C7.2, U4.3 (VI)
- net +12V: now also C20.1, L3.2, U6.4 (FB); no longer C17.1, D11.1 (K)
- net GNDREF: now also C16.2, C19.2, C20.2, D8.2 (A), U6.3 (GND), U6.5 (~{ON}/OFF); no longer C16.1
- net at D1.1 (+), D11.2 (A), D12.1 (K): now also C16.1; no longer C16.2
- new net: D8.1 (K), L3.1, U6.2 (OUT)
- new net VIN: C17.1, C19.1, D11.1 (K), U6.1 (VIN)
Other:
- note removed: "5V"
- moved on the sheet: C16, C7, C8, D3, F1, J4, R5, RV1, U4
