File: Hardware/esp_automation/esp_automation.kicad_pcb (KiCad board)
At the start: 2 copper layers, 119.8 x 99.4 mm, 90 parts, among them J1 UART, J10 Conn_01x02, J11 Conn_01x02, J2 TEMP0, J3 TEMP1, J4 Conn_01x02, J5 Conn_01x02, J6 Conn_01x02, J7 Conn_01x02, J8 Conn_01x02, J9 Conn_01x02, K1 FINDER-32.21-x000, K2 FINDER-32.21-x000, K3 FINDER-32.21-x000, K4 FINDER-32.21-x000, K5 FINDER-32.21-x000, K6 FINDER-32.21-x000, K7 FINDER-32.21-x000, Q1 2N7002, SW1 RESET, SW2 BOOT, T1 Transformer_1P_1S, U1 ESP32-WROOM-32D, U2 ULN2003A, U3 L7805, U4 AMS1117-3.3

Commit message: add software
Connections:
- U1 pad 10: IO25 -> unconnected-(U1-IO25-Pad10)
- U1 pad 11: IO26 -> unconnected-(U1-IO26-Pad11)
- U1 pad 12: IO27 -> unconnected-(U1-IO27-Pad12)
- U1 pad 37: IO23 -> unconnected-(U1-IO23-Pad37)
- U1 pad 8: IO32 -> unconnected-(U1-IO32-Pad8)
- U1 pad 9: IO33 -> unconnected-(U1-IO33-Pad9)
Changed lines of the file:
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@@
   (net 47 "Net-(J4-Pin_1)")
   (net 48 "Net-(U1-IO0)")
-  (net 49 "IO32")
-  (net 50 "IO33")
-  (net 51 "IO25")
-  (net 52 "IO26")
-  (net 53 "IO27")
+  (net 49 "unconnected-(U1-IO32-Pad8)")
+  (net 50 "unconnected-(U1-IO33-Pad9)")
+  (net 51 "unconnected-(U1-IO25-Pad10)")
+  (net 52 "unconnected-(U1-IO26-Pad11)")
+  (net 53 "unconnected-(U1-IO27-Pad12)")
   (net 54 "unconnected-(U1-IO34-Pad6)")
   (net 55 "unconnected-(U1-IO35-Pad7)")
@@
   (net 72 "unconnected-(U1-IO15-Pad23)")
   (net 73 "IO21")
-  (net 74 "IO23")
+  (net 74 "unconnected-(U1-IO23-Pad37)")
   (net 75 "unconnected-(K1-Pad12)")
   (net 76 "Net-(K1-Pad11)")
@@
       (net 55 "unconnected-(U1-IO35-Pad7)") (pinfunction "IO35") (pintype "input+no_connect"))
     (pad "8" smd rect (at -8.75 0.64) (size 1.5 0.9) (layers "F.Cu" "F.Paste" "F.Mask")
-      (net 49 "IO32") (pinfunction "IO32") (pintype "bidirectional"))
+      (net 49 "unconnected-(U1-IO32-Pad8)") (pinfunction "IO32") (pintype "bidirectional+no_connect"))
     (pad "9" smd rect (at -8.75 1.91) (size 1.5 0.9) (layers "F.Cu" "F.Paste" "F.Mask")
-      (net 50 "IO33") (pinfunction "IO33") (pintype "bidirectional"))
+      (net 50 "unconnected-(U1-IO33-Pad9)") (pinfunction "IO33") (pintype "bidirectional+no_connect"))
     (pad "10" smd rect (at -8.75 3.18) (size 1.5 0.9) (layers "F.Cu" "F.Paste" "F.Mask")
-      (net 51 "IO25") (pinfunction "IO25") (pintype "bidirectional"))
+      (net 51 "unconnected-(U1-IO25-Pad10)") (pinfunction "IO25") (pintype "bidirectional+no_connect"))
     (pad "11" smd rect (at -8.75 4.45) (size 1.5 0.9) (layers "F.Cu" "F.Paste" "F.Mask")
-      (net 52 "IO26") (pinfunction "IO26") (pintype "bidirectional"))
+      (net 52 "unconnected-(U1-IO26-Pad11)") (pinfunction "IO26") (pintype "bidirectional+no_connect"))
     (pad "12" smd rect (at -8.75 5.72) (size 1.5 0.9) (layers "F.Cu" "F.Paste" "F.Mask")
-      (net 53 "IO27") (pinfunction "IO27") (pintype "bidirectional"))
+      (net 53 "unconnected-(U1-IO27-Pad12)") (pinfunction "IO27") (pintype "bidirectional+no_connect"))
     (pad "13" smd rect (at -8.75 6.99) (size 1.5 0.9) (layers "F.Cu" "F.Paste" "F.Mask")
       (net 56 "unconnected-(U1-IO14-Pad13)") (pinfunction "IO14") (pintype "bidirectional+no_connect"))
@@
       (net 46 "IO22") (pinfunction "IO22") (pintype "bidirectional"))
     (pad "37" smd rect (at 8.75 -6.98) (size 1.5 0.9) (layers "F.Cu" "F.Paste" "F.Mask")
-      (net 74 "IO23") (pinfunction "IO23") (pintype "bidirectional"))
+      (net 74 "unconnected-(U1-IO23-Pad37)") (pinfunction "IO23") (pintype "bidirectional+no_connect"))
     (pad "38" smd rect (at 8.75 -8.25) (size 1.5 0.9) (layers "F.Cu" "F.Paste" "F.Mask")
       (net 4 "GNDREF") (pinfunction "GND") (pintype "passive"))

Commit message: .
Routing:
- net IO21: track 18.8 -> 21.3 mm
- net IO19: track 16.6 -> 18.6 mm
- net +12V: track 215.6 -> 217.2 mm
- net IO18: track 14.9 -> 16.4 mm
- net IO5: track 13.2 -> 14.3 mm
- net IO17: track 11.5 -> 12.2 mm
- net Net-(T1-SA): track 26.2 -> 25.7 mm
- net GNDREF: vias 9 -> 68
Other:
- outline, holes or cut-outs redrawn

Commit message: .
Parts:
- removed C6: 220UF 25V, Capacitor_SMD:CP_Elec_8x10.5
- removed R4: 330R, Resistor_SMD:R_0805_2012Metric
- removed U3: L7805, Package_TO_SOT_SMD:TO-252-2
- added C19: 100nF, Capacitor_SMD:C_0805_2012Metric, F.Cu at (192.0, 71.5)
- added C23: 1000UF 25V SMD, Capacitor_SMD:CP_Elec_10x12.6, F.Cu at (183.6, 76.5)
- added D15: SS34, Diode_SMD:D_SMC, F.Cu at (176.0, 56.5)
- added L1: 100uH, Inductor_SMD:L_12x12mm_H4.5mm, F.Cu at (188.0, 59.9)
- added U5: LM2576HVS-12, Package_TO_SOT_SMD:TO-263-5_TabPin3, F.Cu at (205.9, 59.6)
- D1: footprint Package_TO_SOT_SMD:TO-269AA -> GOFootprint:DB157S
- D2: value Led_Blue -> SM712_SOT23; footprint LED_SMD:LED_0805_2012Metric -> Package_TO_SOT_SMD:SOT-23
- T1: footprint gkhnmlym:ASLAN220-12VAC -> GOFootprint:ASLAN 151112
- moved D2 27.8 mm to (156.9, 61.9), turned to -135 degrees
- moved RV1 18.7 mm to (206.6, 143.9), turned to 90 degrees
- moved D12 15.9 mm to (217.9, 72.6), turned to 90 degrees
- moved T1 12.7 mm to (175.4, 130.2)
- moved C4 12.5 mm to (202.2, 134.8)
- moved H2 12.0 mm to (217.2, 57.7)
- moved H4 12.0 mm to (217.2, 146.3)
- moved C5 11.4 mm to (215.6, 89.6)
- moved D11 11.1 mm to (204.1, 72.6), turned to -90 degrees
- moved D1 10.9 mm to (202.3, 78.6)
- moved C16 10.9 mm to (211.0, 72.2), turned to 90 degrees
- moved D3 10.1 mm to (172.6, 74.5), turned to 90 degrees
- moved C7 9.77 mm to (177.5, 66.8), turned to -90 degrees
- moved C17 9.47 mm to (197.1, 73.2), turned to -90 degrees
- moved R5 8.26 mm to (172.6, 70.9), turned to 90 degrees
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Connections:
- BZ1 pad 1: +5V -> +12V
- C16 pad 1: GNDREF -> Net-(D1-+)
- C16 pad 2: Net-(D1-+) -> GNDREF
- C17 pad 1: +12V -> VIN
- C7 pad 2: +5V -> +12V
- D11 pad 1: +12V -> VIN
- D2 pad 1: GNDREF -> RXD0
- D2 pad 2: Net-(D2-A) -> TXD0
- U4 pad 3: +5V -> +12V
Routing:
- net +5V: track 54.7 -> 0.00 mm
- net VIN: track 0.00 -> 30.7 mm, vias 0 -> 2
- net Net-(D15-K): track 0.00 -> 20.8 mm
- net L: track 22.9 -> 39.0 mm
- net Net-(T1-SA): track 25.7 -> 36.9 mm
- net Net-(T1-SB): track 16.2 -> 25.9 mm
- net +3V3: track 134.1 -> 124.6 mm, vias 2 -> 3
- net Net-(D1-+): track 21.5 -> 26.9 mm
- net N: track 209.4 -> 214.7 mm
- net Net-(D2-A): track 1.81 -> 0.00 mm
- net GNDREF: track 4.21 -> 5.63 mm, vias 68 -> 11
- net Net-(J4-Pin_1): track 9.33 -> 7.93 mm
- net +12V: track 217.2 -> 216.1 mm
Other:
- board size 119.8 x 99.4 mm -> 131.7 x 99.4 mm
