File: Hardware/esp_automation/esp_automation.kicad_sch (KiCad schematic)
At the start: 12 parts, among them J1 UART, SW1 RESET, SW2 BOOT, U1 ESP32-WROOM-32D

Commit message: add software
Connections:
- net IO23: no longer names the net of U1.37 (IO23)
- net IO25: no longer names the net of U1.10 (IO25)
- net IO26: no longer names the net of U1.11 (IO26)
- net IO27: no longer names the net of U1.12 (IO27)
- net IO32: no longer names the net of U1.8 (IO32)
- net IO33: no longer names the net of U1.9 (IO33)
- no-connect marks 12 -> 18
Other:
- moved on the sheet: C1, C2, C3, J1, R1, SW1, SW2, U1

Commit message: .
Parts:
- added D2: SM712_SOT23, Package_TO_SOT_SMD:SOT-23, symbol Diode:SM712_SOT23
Connections:
- net GNDREF: now also D2.3 (common)
- net RXD0: now also D2.1 (A1)
- net TXD0: now also D2.2 (A2)
Changed lines of the file:
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@@
+    )
+  )
+  (global_label "RXD0" (shape input) (at 23.495 98.425 180) (fields_autoplaced)
+    (effects (font (size 1.27 1.27)) (justify right))
+    (property "Intersheetrefs" "${INTERSHEET_REFS}" (at 15.6302 98.425 0)
+      (effects (font (size 1.27 1.27)) (justify right) hide)
     )
   )
@@
     (effects (font (size 1.27 1.27)) (justify left))
     (property "Intersheetrefs" "${INTERSHEET_REFS}" (at 22.1456 21.4448 90)
+      (effects (font (size 1.27 1.27)) (justify left) hide)
+    )
+  )
+  (global_label "TXD0" (shape input) (at 41.275 98.425 0) (fields_autoplaced)
+    (effects (font (size 1.27 1.27)) (justify left))
+    (property "Intersheetrefs" "${INTERSHEET_REFS}" (at 48.8374 98.425 0)
       (effects (font (size 1.27 1.27)) (justify left) hide)
     )
@@
     )
   )
+  (symbol (lib_id "power:GNDREF") (at 32.385 102.235 0) (unit 1)
+    (in_bom yes) (on_board yes) (dnp no) (fields_autoplaced)
+    (property "Reference" "#PWR020" (at 32.385 108.585 0)
+      (effects (font (size 1.27 1.27)) hide)
+    )
+    (property "Value" "GNDREF" (at 34.925 103.5049 0)
+      (effects (font (size 1.27 1.27)) (justify left))
+    )
+    (property "Footprint" "" (at 32.385 102.235 0)
+      (effects (font (size 1.27 1.27)) hide)
+    )
+    (property "Datasheet" "" (at 32.385 102.235 0)
+      (effects (font (size 1.27 1.27)) hide)
+    )
+    (pin "1")
+    (instances
+      (project "esp_automation"
+        (path "/beacb42a-3344-450f-9913-7e99b3038b5c"
+          (reference "#PWR020") (unit 1)
+        )
+      )
+    )
+  )
   (symbol (lib_id "Mechanical:MountingHole") (at 243.84 62.23 0) (unit 1)
     (in_bom yes) (on_board yes) (dnp no) (fields_autoplaced)
@@
         )
       )
+    )
+  )
+  (symbol (lib_id "Diode:SM712_SOT23") (at 32.385 98.425 0) (unit 1)
+    (in_bom yes) (on_board yes) (dnp no) (fields_autoplaced)
+    (property "Reference" "D2" (at 32.385 93.345 0)
+      (effects (font (size 1.27 1.27)))
+    )
+    (property "Value" "SM712_SOT23" (at 32.385 95.885 0)
+      (effects (font (size 1.27 1.27)))
+    )
+    (property "Footprint" "Package_TO_SOT_SMD:SOT-23" (at 32.385 107.315 0)
+      (effects (font (size 1.27 1.27)) hide)
+    )
+    (property "Datasheet" "https://www.littelfuse.com/~/media/electronics/datasheets/tvs_diode_arrays/littelfuse_tvs_diode_array_sm712_datasheet.pdf.pdf" (at 28.575 98.425 0)
+      (effects (font (size 1.27 1.27)) hide)
+    )
+    (pin "1")
+    (pin "2")
+    (pin "3")
+    (instances
+      (project "esp_automation"
+        (path "/beacb42a-3344-450f-9913-7e99b3038b5c"
+          (reference "D2") (unit 1)
+        )
+      )
